Commit message: Added database folder to use soft hand outside ros in gazebo. Added new mesh of palm

File: model/complete_soft_hand.urdf.xacro (robot description, xacro)
@@ -281,5 +281,6 @@
 				<origin xyz="0 0 0" rpy="0 0 0" />
 				<geometry>
-					<mesh filename="package://complete_soft_hand/meshes/palm_hand.stl" scale=" .001 .001 .001" />
+					<!-- <mesh filename="package://complete_soft_hand/meshes/palm_hand.stl" scale=" .001 .001 .001" /> -->
+					<mesh filename="package://complete_soft_hand/meshes/palm_hand2.stl" scale=" .001 .001 .001" />
 				</geometry>
 				<material name="LightGrey" />
